File: Strain Wave Motor Control Board.kicad_pcb (KiCad board)
At the start: 2 copper layers, 72 parts, among them J3 Screw_Terminal_01x02, J4 Conn_01x03_Socket, Q1 CSD18531Q5A, Q3 CSD18531Q5A, Q7 NMOS, Q8 NMOS, U1 HUSB238A-xxxxx-QN16R, U3 LTC4007, U4 LM2596S-5, U5 SN74LVC1T45DCK, U7 Optocoupler_DC_PhotoNPN_AKEC, U8 Optocoupler_DC_PhotoNPN_AKEC

Commit message: ESP32 schematic added
Parts:
- removed J3: Screw_Terminal_01x02, TerminalBlock:TerminalBlock_MaiXu_MX126-5.0-02P_1x02_P5.00mm
- removed J4: Conn_01x03_Socket, Connector_PinSocket_2.54mm:PinSocket_1x03_P2.54mm_Vertical
- removed Q7, Q8: NMOS, Package_TO_SOT_SMD:TO-263-2
- removed R34: 10K, Resistor_SMD:R_0805_2012Metric_Pad1.20x1.40mm_HandSolder
- removed R35, R36: 750, Resistor_SMD:R_0805_2012Metric_Pad1.20x1.40mm_HandSolder
- removed U7, U8: Optocoupler_DC_PhotoNPN_AKEC, Package_DIP:DIP-4_W7.62mm_SMDSocket_SmallPads
- added D1: MBRS130T3G, MBRS130T3G:DIOM5436X247N, F.Cu at (96.8, 89.4)
- added J1: GSB1C41110SSHR, GSB1C41110SSHR:AMPHENOL_GSB1C41110SSHR, F.Cu at (118.3, 44.6)
- added J2: S4B-XH-SM4-TB, S4B_XH_SM4_TB:JST_S4B-XH-SM4-TB, F.Cu at (129.2, 85.3)
- added Q2: AO4407A, AO4407A:SOIC127P600X175-8N, F.Cu at (116.4, 65.8)
- added Q4: AO4407A, AO4407A:SOIC127P600X175-8N, F.Cu at (116.4, 72.3)
- added Q5: SI4178DY-T1-GE3, SI4178DY-T1-GE3:SOIC_Y-T1-GE3_VIS, F.Cu at (116.0, 85.5)
- added Q6: AO4407A, AO4407A:SOIC127P600X175-8N, F.Cu at (116.4, 78.9)
- added TH1: Thermistor_NTC 10k, Resistor_SMD:R_0402_1005Metric_Pad0.72x0.64mm_HandSolder, F.Cu at (143.3, 40.0)
- added U2: BQ7791500PWR, BQ7791500PWR:PW24_TEX, F.Cu at (137.0, 43.8)
- TH2: value 10k -> Thermistor_NTC 10k; footprint Resistor_SMD:R_0805_2012Metric_Pad1.20x1.40mm_HandSolder -> Resistor_SMD:R_0402_1005Metric_Pad0.72x0.64mm_HandSolder
- U5: value SN74LVC1T45DCK -> ESP32-C6; footprint Package_TO_SOT_SMD:SOT-363_SC-70-6_Handsoldering -> ESP32-C6:E
- moved R27 63.2 mm to (109.3, 40.5)
- moved R18 58.5 mm to (104.5, 40.5)
- moved R19 58.5 mm to (104.5, 43.4)
- moved R20 58.5 mm to (104.5, 46.4)
- moved R10 54.0 mm to (99.8, 43.4)
- moved R11 54.0 mm to (99.8, 46.4)
- moved R9 54.0 mm to (99.8, 40.5)
- moved R12 54.0 mm to (99.8, 49.3)
- moved R13 54.0 mm to (99.8, 52.3)
- moved R32 51.6 mm to (109.3, 55.2)
- moved R28 51.6 mm to (109.3, 43.4)
- moved R29 51.6 mm to (109.3, 46.4)
- moved R30 51.6 mm to (109.3, 49.3)
- moved R31 51.6 mm to (109.3, 52.3)
- moved R33 51.6 mm to (109.3, 58.2)
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Connections:
- net 'CHG renamed /Power Supply/~CHG
- net 'FAULT renamed /Power Supply/~FAULT
- net 'FLAG renamed /Power Supply/~FLAG
- net 'Icl renamed /Power Supply/~ICL
- net 'LOBAT renamed /Power Supply/~LOBAT
- net 5V_OUT renamed /Power Supply/5V
- net ACP renamed /Power Supply/ACP
- net PRES renamed /Power Supply/PRES
- net SHDN renamed /Power Supply/SHDN
- net VLOGIC renamed /Power Supply/VLOGIC
- C10 pad 2: DC_GND -> GND
- C11 pad 1: DC_GND -> GND
- C12 pad 1: DC_GND -> GND
- C13 pad 2: DC_GND -> GND
- C14 pad 2: DC_GND -> GND
- C16 pad 2: DC_GND -> GND
- C17 pad 1: DC_GND -> GND
- C18 pad 2: DC_GND -> GND
- C19 pad 2: DC_GND -> GND
- C3 pad 2: DC_GND -> GND
- C4 pad 1: DC_GND -> GND
- C5 pad 2: DC_GND -> GND
- C6 pad 1: DC_GND -> GND
- C7 pad 2: DC_GND -> GND
- C9 pad 2: DC_GND -> GND
- D2 pad 2: DC_GND -> GND
- R11 pad 2: DC_GND -> GND
- R12 pad 2: DC_GND -> GND
- R20 pad 2: DC_GND -> GND
- R26 pad 2: DC_GND -> GND
- R29 pad 2: DC_GND -> GND
- R5 pad 1: DC_GND -> GND
- R6 pad 2: DC_GND -> GND
- R8 pad 2: DC_GND -> GND
- TH2 pad 1: DC_GND -> GND
- U1 pad 12: DC_GND -> GND
- U1 pad 17: DC_GND -> GND
- U3 pad 21: DC_GND -> GND
- U3 pad 6: DC_GND -> GND
- U3 pad 7: DC_GND -> GND
- U4 pad 3: DC_GND -> GND
- U4 pad 5: DC_GND -> GND
- U5 pad 1: /Control System/H-Bridge/3V3 -> unconnected-(U5-3.3V-Pad1)
- U5 pad 2: DC_GND -> unconnected-(U5-RST-Pad2)
- U5 pad 3: /Control System/H-Bridge/EN -> unconnected-(U5-GPIO4-Pad3)
- U5 pad 4: Net-(U5-B) -> unconnected-(U5-GPIO5-Pad4)
- U5 pad 5: /Control System/H-Bridge/3V3 -> unconnected-(U5-GPIO6-Pad5)
- U5 pad 6: /Control System/H-Bridge/5V -> unconnected-(U5-GPIO7-Pad6)

Commit message: started layout
Parts:
- added D4: 1655, 1655:LED_1655, F.Cu at (150.6, 131.8)
- added J3: RJHSE-5080, RJ45:CONN_RJSBE5080_16P13X12P57_AMP, F.Cu at (146.4, 58.6)
- added J4: ~, Battery_Connector:LiPo Wire Pads, F.Cu at (132.5, 136.5)
- added S1: 100SP1T1B4M2QE, Switches:SW_100SP1T1B4M2QE, F.Cu at (128.0, 131.9)
- added S2: 100SP1T1B4M2QE, Switches:SW_100SP1T1B4M2QE, F.Cu at (136.0, 131.9)
- added U6: SN74LVC1T45DCK, Package_TO_SOT_SMD:SOT-363_SC-70-6, F.Cu at (157.2, 131.5)
- C9, R10, R7: moved to B.Cu
- D2, D3: value 1N5822 -> MBRS130T3G; footprint Diode_THT:D_DO-201AD_P15.24mm_Horizontal -> MBRS130T3G:DIOM5436X247N
- moved TH1 118.9 mm to (26.2, 60.4)
- moved TH2 118.9 mm to (26.2, 62.4)
- moved Q1 107.1 mm to (28.7, 49.4)
- moved Q3 107.1 mm to (28.7, 56.1)
- moved J1 100.7 mm to (114.9, 145.2)
- moved R10 90.7 mm to (108.0, 133.8), turned to 90 degrees
- moved R11 86.2 mm to (114.8, 131.2), turned to 180 degrees
- moved R12 82.7 mm to (111.0, 131.2), turned to 180 degrees
- moved R7 82.5 mm to (118.5, 140.2), turned to 180 degrees
- moved D1 71.9 mm to (71.1, 22.2)
- moved L2 70.8 mm to (27.0, 21.0)
- moved R1 70.8 mm to (27.0, 23.9)
- moved R13 70.8 mm to (31.7, 32.8)
- moved R14 70.8 mm to (31.7, 35.7)
- moved R16 70.8 mm to (31.7, 41.6)
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Connections:
- net /Power Supply/BATT+ renamed /Power Supply/CELL_3
- C19 pad 1: /Power Supply/5V -> /5V
- C5 pad 1: Net-(U2-VDD) -> /Power Supply/PRES
- J1 pad A4_B9: /Power Supply/VBUS -> /Power Supply/USB_VBUS
- J1 pad B4_A9: /Power Supply/VBUS -> /Power Supply/USB_VBUS
- J2 pad 4: /Power Supply/BATT- -> GND
- L2 pad 1: /Power Supply/5V -> /5V
- Q3 pad 1: /Power Supply/BATT- -> /Power Supply/PACK-
- Q3 pad 2: /Power Supply/BATT- -> /Power Supply/PACK-
- Q3 pad 3: /Power Supply/BATT- -> /Power Supply/PACK-
- R1 pad 2: Net-(U2-VDD) -> /Power Supply/PRES
- R17 pad 2: /Power Supply/BATT- -> /Power Supply/PACK-
- R21 pad 2: /Power Supply/BATT- -> /Power Supply/PACK-
- R22 pad 1: /Power Supply/ACP -> /ACP
- R22 pad 2: /Power Supply/VLOGIC -> /VLOGIC
- R23 pad 1: /Power Supply/~FAULT -> /~FAULT
- R23 pad 2: /Power Supply/VLOGIC -> /VLOGIC
- R25 pad 1: /Power Supply/~FLAG -> /~FLAG
- R25 pad 2: /Power Supply/VLOGIC -> /VLOGIC
- U2 pad 1: Net-(U2-VDD) -> /Power Supply/PRES
- U2 pad 16: GND -> unconnected-(U2-CBI-Pad16)
- U2 pad 20: unconnected-(U2-CCFG-Pad20) -> GND
- U2 pad 3: unconnected-(U2-VC5-Pad3) -> Net-(U2-VC3)
- U2 pad 4: unconnected-(U2-VC4-Pad4) -> Net-(U2-VC3)
- U3 pad 13: /Power Supply/~ICL -> /~ICL
- U3 pad 17: /Power Supply/~FLAG -> /~FLAG
- U3 pad 2: /Power Supply/~CHG -> /~CHG
- U3 pad 24: /Power Supply/SHDN -> /SHDN
- U3 pad 3: /Power Supply/ACP -> /ACP
- U3 pad 5: /Power Supply/~FAULT -> /~FAULT
- U3 pad 8: /Power Supply/~LOBAT -> /~LOBAT
- U4 pad 4: /Power Supply/5V -> /5V
- U5 pad 1: unconnected-(U5-3.3V-Pad1) -> /VLOGIC
- U5 pad 10: unconnected-(U5-GPIO10-Pad10) -> /~LOBAT
- U5 pad 11: unconnected-(U5-GPIO11-Pad11) -> /ACP
- U5 pad 12: unconnected-(U5-GPIO2-Pad12) -> /CTRL_1
- U5 pad 13: unconnected-(U5-GPIO3-Pad13) -> /CTRL_2
- U5 pad 14: unconnected-(U5-5V-Pad14) -> /5V
- U5 pad 15: unconnected-(U5-GND-Pad15) -> GND
- U5 pad 17: unconnected-(U5-GND-Pad17) -> GND
- U5 pad 20: unconnected-(U5-GPIO15-Pad20) -> /GPIO_X
- U5 pad 3: unconnected-(U5-GPIO4-Pad3) -> /CTRL_3
- U5 pad 31: unconnected-(U5-GND-Pad31) -> GND
- U5 pad 4: unconnected-(U5-GPIO5-Pad4) -> /SHDN
- U5 pad 5: unconnected-(U5-GPIO6-Pad5) -> /PRES
- U5 pad 6: unconnected-(U5-GPIO7-Pad6) -> /~CHG
- U5 pad 7: unconnected-(U5-GPIO0-Pad7) -> /~FAULT
- U5 pad 8: unconnected-(U5-GPIO1-Pad8) -> /~FLAG
- U5 pad 9: unconnected-(U5-GPIO8-Pad9) -> /~ICL
Routing:
- net /Power Supply/VBUS: track 0.00 -> 67.5 mm, vias 0 -> 1
- net /Power Supply/USB_VBUS: track 0.00 -> 38.6 mm, vias 0 -> 1
- net /VLOGIC: track 0.00 -> 30.2 mm, vias 0 -> 2
- net /5V: track 0.00 -> 16.9 mm, vias 0 -> 1
- net /Power Supply/PACK+: track 0.00 -> 15.9 mm
- net Net-(D4-DIN): track 0.00 -> 11.3 mm
- net /Power Supply/D-: track 0.00 -> 9.81 mm, vias 0 -> 2
- net /Power Supply/D+: track 0.00 -> 7.56 mm, vias 0 -> 2
- net Net-(U1-VDD): track 0.00 -> 7.42 mm, vias 0 -> 1
- net Net-(Q2-Pad4): track 0.00 -> 6.68 mm, vias 0 -> 1
- net Net-(U1-GATE): track 0.00 -> 5.45 mm, vias 0 -> 1
- net /Power Supply/CC1: track 0.00 -> 5.25 mm
- net /Power Supply/CC2: track 0.00 -> 5.07 mm
- net Net-(U1-SCL/SNK_ISET): track 0.00 -> 4.14 mm
- net Net-(U1-SDA/SNK_VSET): track 0.00 -> 3.01 mm
Other:
- board outline added: 100 x 100 mm

Commit message: done
Parts:
- removed L1: 10uH, Inductor_SMD:L_0805_2012Metric_Pad1.05x1.20mm_HandSolder
- removed L2: 33uH, Inductor_SMD:L_0805_2012Metric_Pad1.15x1.40mm_HandSolder
- added L3: NR6045T100M, NR6045T100M:IND_NR6045T100M, F.Cu at (193.0, 84.5)
- added L4: SRN8040-330M, SRN8040:IND_BOURNS_SRN8040, F.Cu at (121.5, 107.5)
- C1, C10, C11, C13, C2, C3, C7, C8: footprint Capacitor_SMD:C_0805_2012Metric_Pad1.18x1.45mm_HandSolder -> LED_SMD:LED_0805_2012Metric_Pad1.15x1.40mm_HandSolder; moved to B.Cu
- C12, C4: footprint Capacitor_SMD:C_0805_2012Metric_Pad1.18x1.45mm_HandSolder -> LED_SMD:LED_0805_2012Metric_Pad1.15x1.40mm_HandSolder
- C14, C5, C6: footprint Capacitor_SMD:C_0805_2012Metric_Pad1.18x1.45mm_HandSolder -> Capacitor_SMD:C_0603_1608Metric_Pad1.08x0.95mm_HandSolder; moved to B.Cu
- C15, C9: footprint Capacitor_SMD:C_0805_2012Metric_Pad1.18x1.45mm_HandSolder -> Capacitor_SMD:C_0603_1608Metric_Pad1.08x0.95mm_HandSolder
- C16: value 680uF -> UCL1E681MNL1GS; footprint Capacitor_SMD:C_0805_2012Metric_Pad1.18x1.45mm_HandSolder -> 680:CAPAE1030X1350N
- C19: footprint Capacitor_SMD:C_0805_2012Metric_Pad1.18x1.45mm_HandSolder -> Capacitor_SMD:C_1206_3216Metric_Pad1.33x1.80mm_HandSolder
- R13: value 4.5k -> 4k
- R18, R19, R20, R22, R23, R24, R25, R26, R27, R29, R6, R8, R9, TH1, TH2: moved to B.Cu
- R30: value 0.033 -> 0.025
- R32: value 3.01k -> 0.025
- moved R31 162.4 mm to (197.5, 77.0), turned to 90 degrees
- moved R27 159.8 mm to (181.0, 98.5)
- moved R32 158.3 mm to (194.0, 77.0), turned to 90 degrees
- moved R28 155.3 mm to (181.0, 91.5), turned to 90 degrees
- moved R33 152.9 mm to (189.5, 76.0), turned to 180 degrees
- moved R29 152.8 mm to (174.5, 101.5)
- moved C13 147.7 mm to (183.0, 102.0)
- moved R30 146.9 mm to (178.0, 83.5), turned to 90 degrees
- moved C15 146.5 mm to (181.5, 96.0), turned to 180 degrees
- moved C18 145.8 mm to (195.0, 73.0)
- moved R26 145.3 mm to (174.0, 91.5), turned to 90 degrees
- moved R23 144.3 mm to (168.0, 95.0), turned to 180 degrees
- moved R25 144.3 mm to (168.0, 100.9), turned to 180 degrees
- moved R22 144.3 mm to (168.0, 92.0), turned to 180 degrees
- moved D1 142.0 mm to (195.0, 91.5), turned to -90 degrees
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- renumbered S2 to S3
Connections:
- J3 pad 7: /CRTL_3 -> /CTRL_3
- R13 pad 1: Net-(R13-Pad1) -> Net-(Q1-G)
- R14 pad 1: Net-(R13-Pad1) -> Net-(Q1-G)
- R14 pad 2: Net-(Q1-G) -> Net-(Q1-S-Pad1)
- U5 pad 21: unconnected-(U5-GPIO23-Pad21) -> /Power Supply/NEOPIXEL
Routing:
- net /Power Supply/CELL_3: track 0.00 -> 253.9 mm, vias 0 -> 4
- net /Power Supply/CELL_2: track 0.00 -> 142.2 mm, vias 0 -> 2
- net /Power Supply/CELL_1: track 0.00 -> 140.9 mm, vias 0 -> 2
- net /5V: track 16.9 -> 141.2 mm, vias 1 -> 4
- net /Power Supply/PACK-: track 0.00 -> 117.8 mm, vias 0 -> 2
- net /Power Supply/12V: track 0.00 -> 103.6 mm, vias 0 -> 5
- net /GPIO_X: track 0.00 -> 99.8 mm, vias 0 -> 2
- net /CTRL_1: track 0.00 -> 98.0 mm, vias 0 -> 1
- net /CTRL_2: track 0.00 -> 82.7 mm, vias 0 -> 2
- net /CTRL_3: track 0.00 -> 63.0 mm, vias 0 -> 2
- net /ACP: track 0.00 -> 56.0 mm, vias 0 -> 1
- net /Power Supply/NEOPIXEL: track 0.12 -> 47.9 mm
- net /~LOBAT: track 0.00 -> 43.8 mm, vias 0 -> 1
- net /Power Supply/CSP: track 0.00 -> 40.6 mm
- net /~CHG: track 0.00 -> 40.5 mm
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- added copper zone on B.Cu, net GND
- added copper zone on F.Cu, net GND
