File: Strain Wave Motor Control Board.kicad_sch (KiCad schematic)
At the start: 0 parts

Commit message: added sub-schematics
Other:
- added sheet Control System (control_system.kicad_sch)
- added sheet Power Supply (power_supply.kicad_sch)
Changed lines of the file:
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@@
 	(generator_version "9.0")
 	(paper "A4")
+	(sheet
+		(at 60.96 31.75)
+		(size 48.26 26.67)
+		(exclude_from_sim no)
+		(in_bom yes)
+		(on_board yes)
+		(dnp no)
+		(fields_autoplaced yes)
+		(stroke
+			(width 0.1524)
+			(type solid)
+		)
+		(fill
+			(color 0 0 0 0.0000)
+		)
+		(property "Sheetname" "Power Supply"
+			(at 60.96 31.0384 0)
+			(effects
+				(font
+					(size 1.27 1.27)
+				)
+				(justify left bottom)
+			)
+		)
+		(property "Sheetfile" "power_supply.kicad_sch"
+			(at 60.96 59.0046 0)
+			(effects
+				(font
+					(size 1.27 1.27)
+				)
+				(justify left top)
+			)
+		)
+		(instances
+			(project "Strain Wave Motor Control Board"
+				(path "/6a10ea30-147f-4e88-a5c3-bf0fd41178aa"
+					(page "2")
+				)
+			)
+		)
+	)
+	(sheet
+		(at 151.13 31.75)
+		(size 50.8 27.94)
+		(exclude_from_sim no)
+		(in_bom yes)
+		(on_board yes)
+		(dnp no)
+		(fields_autoplaced yes)
+		(stroke
+			(width 0.1524)
+			(type solid)
+		)
+		(fill
+			(color 0 0 0 0.0000)
+		)
+		(property "Sheetname" "Control System"
+			(at 151.13 31.0384 0)
+			(effects
+				(font
+					(size 1.27 1.27)
+				)
+				(justify left bottom)
+			)
+		)
+		(property "Sheetfile" "control_system.kicad_sch"
+			(at 151.13 60.2746 0)
+			(effects
+				(font
+					(size 1.27 1.27)
+				)
+				(justify left top)
+			)
+		)
+		(instances
+			(project "Strain Wave Motor Control Board"
+				(path "/6a10ea30-147f-4e88-a5c3-bf0fd41178aa"
+					(page "3")
+				)
+			)
+		)
+	)
 	(sheet_instances
 		(path "/"

Commit message: ESP32 schematic added
Parts:
- added U5: ESP32-C6, ESP32-C6:E, symbol SWM Components:ESP32-C6
Other:
- removed sheet Control System
Changed lines of the file:
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@@
 	(generator_version "9.0")
 	(paper "A4")
+	(symbol
+		(lib_id "SWM Components:ESP32-C6")
+		(at 91.44 91.44 0)
+		(unit 1)
+		(exclude_from_sim no)
+		(in_bom yes)
+		(on_board yes)
+		(dnp no)
+		(fields_autoplaced yes)
+		(property "Reference" "U5"
+			(at 91.44 87.63 0)
+			(effects
+				(font
+					(size 1.27 1.27)
+				)
+			)
+		)
+		(property "Value" "ESP32-C6"
+			(at 91.44 90.17 0)
+			(effects
+				(font
+					(size 1.27 1.27)
+				)
+			)
+		)
+		(property "Footprint" "ESP32-C6:E"
+			(at 91.44 91.44 0)
+			(effects
+				(font
+					(size 1.27 1.27)
+				)
+				(hide yes)
+			)
+		)
+		(property "Datasheet" ""
+			(at 91.44 91.44 0)
+			(effects
+				(font
+					(size 1.27 1.27)
+				)
+				(hide yes)
+			)
+		)
+		(property "Description" ""
+			(at 91.44 91.44 0)
+			(effects
+				(font
+					(size 1.27 1.27)
+				)
+				(hide yes)
+			)
+		)
+		(pin "32"
+		)
+		(pin "12"
+		)
+		(pin "5"
+		)
+		(pin "26"
+		)
+		(pin "15"
+		)
+		(pin "8"
+		)
+		(pin "14"
+		)
+		(pin "28"
+		)
+		(pin "25"
+		)
+		(pin "2"
+		)
+		(pin "20"
+		)
+		(pin "11"
+		)
+		(pin "3"
+		)
+		(pin "13"
+		)
+		(pin "21"
+		)
+		(pin "18"
+		)
+		(pin "19"
+		)
+		(pin "4"
+		)
+		(pin "17"
+		)
+		(pin "6"
+		)
+		(pin "7"
+		)
+		(pin "9"
+		)
+		(pin "16"
+		)
+		(pin "10"
+		)
+		(pin "1"
+		)
+		(pin "31"
+		)
+		(pin "22"
+		)
+		(pin "30"
+		)
+		(pin "27"
+		)
+		(pin "24"
+		)
+		(pin "29"
+		)
+		(pin "23"
+		)
+		(instances
+			(project ""
+				(path "/6a10ea30-147f-4e88-a5c3-bf0fd41178aa"
+					(reference "U5")
+					(unit 1)
+				)
+			)
+		)
+	)
 	(sheet
 		(at 60.96 31.75)
@@
 				)
 			)
-		)
-	)
-	(sheet
-		(at 151.13 31.75)
-		(size 50.8 27.94)
-		(exclude_from_sim no)
-		(in_bom yes)
-		(on_board yes)
-		(dnp no)
-		(fields_autoplaced yes)
-		(stroke
-			(width 0.1524)
-			(type solid)
-		)
-		(fill
-			(color 0 0 0 0.0000)
-		)
-		(property "Sheetname" "Control System"
-			(at 151.13 31.0384 0)
-			(effects
-				(font
-					(size 1.27 1.27)
-				)
-				(justify left bottom)
-			)
-		)
-		(property "Sheetfile" "control_system.kicad_sch"
-			(at 151.13 60.2746 0)
-			(effects
-				(font
-					(size 1.27 1.27)
-				)
-				(justify left top)
-			)
-		)
-		(instances
-			(project "Strain Wave Motor Control Board"
-				(path "/6a10ea30-147f-4e88-a5c3-bf0fd41178aa"
-					(page "3")
-				)
-			)

Commit message: started layout
Parts:
- added J3: RJHSE-5080, CONN_RJSBE5080_16P13X12P57_AMP, symbol RJ45:RJHSE-5080
Connections:
- net VLOGIC: now reaches U5.1 (3.3V)
- net ~LOBAT: now reaches U5.10 (GPIO10)
- net ACP: now reaches U5.11 (GPIO11)
- net CTRL_1: now reaches U5.12 (GPIO2)
- net CTRL_1: now also J3.5
- net CTRL_2: now reaches U5.13 (GPIO3)
- net CTRL_2: now also J3.6
- net 5V: now reaches U5.14 (5V)
- net 5V: now also J3.1, J3.2
- net GND: now reaches U5.15 (GND)
- net GND: now also U5.17 (GND), U5.31 (GND), J3.3, J3.4
- net GPIO_X: now reaches U5.20 (GPIO15)
- net GPIO_X: now also J3.8
- net CTRL_3: now reaches U5.3 (GPIO4)
- net SHDN: now reaches U5.4 (GPIO5)
- net PRES: now reaches U5.5 (GPIO6)
- net ~CHG: now reaches U5.6 (GPIO7)
- net ~FAULT: now reaches U5.7 (GPIO0)
- net ~FLAG: now reaches U5.8 (GPIO1)
- net ~ICL: now reaches U5.9 (GPIO8)
- new net CRTL_3: J3.7
Other:
- sheet Power Supply ports: added 5V, ACP, GND, PRES, SHDN, VLOGIC, ~CHG, ~FAULT, ~FLAG, ~ICL, ~LOBAT; removed none

Commit message: done
Connections:
- net CRTL_3 is gone; now on net CTRL_3: J3.7
- net Power Supply/NEOPIXEL: now reaches U5.21 (GPIO23)
Other:
- sheet Power Supply ports: added NEOPIXEL; removed none
Changed lines of the file:
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@@
+	(wire
+		(pts
+			(xy 90.17 58.42) (xy 90.17 104.14)
+		)
+		(stroke
+			(width 0)
+			(type default)
+		)
+	)
 	(wire
 		(pts
@@
 	(wire
 		(pts
-			(xy 165.1 33.02) (xy 177.8 33.02)
+			(xy 90.17 104.14) (xy 101.6 104.14)
 		)
 		(stroke
@@
 		)
 	)
+	(wire
+		(pts
+			(xy 165.1 33.02) (xy 177.8 33.02)
+		)
+		(stroke
+			(width 0)
+			(type default)
+		)
+	)
 	(label "CTRL_2"
 		(at 63.5 124.46 0)
@@
 		)
 	)
-	(label "CRTL_3"
+	(label "CTRL_3"
 		(at 165.1 40.64 0)
 		(effects
@@
 			(effects
 				(font
+					(size 1.27 1.27)
+				)
+				(justify left)
+			)
+		)
+		(pin "NEOPIXEL" input
+			(at 90.17 58.42 270)
+			(effects
+				(font
